Commit message: REFACTOR-001: plant_params.yaml single source + hard stale-gain failure
double_pendulum.urdf.xacro and linear_model.py's PendulumParams each
hardcoded their own independent copy of m1/m2/L1/L2/damping/torque-limit
values, with nothing enforcing they stayed in sync -- exactly the risk
SKILL-CONTROL-MODEL-CONSISTENCY (a REJECTed candidate, never promoted to
active) was written to guard against as a remembered procedure.

Now both sides read double_pendulum_description/config/plant_params.yaml
directly: the xacro via a native xacro.load_yaml() call (found by
reading the xacro package source -- no custom code-generation step
needed), Python via a new shared plant_params.py loader + hash function.

Also added a hard runtime check: design_lqr_gains.py precomputes and
caches the LQR gain keyed by plant_hash+Q/R weights; lqr_node.py loads
that cache and REFUSES to start on any mismatch (STALE GAIN error, exit
1) instead of silently computing a fresh-but-undetected-as-different
gain or using a stale one. Verified directly: editing plant_params.yaml
without regenerating the cache produces the exact expected error;
regenerating it restores normal startup. Side benefit: lqr_node.py
startup dropped from ~54s (CARE solve every time) to ~3s (cache hit).

Two real xacro bugs hit and fixed along the way:  doesn't
nest inside a ${} Python-eval block (switched to a path relative to the
xacro file's own directory), and XML comments can't contain a literal
-- anywhere (broke on my own comment text, reworded).

Retired SKILL-CONTROL-MODEL-CONSISTENCY with reasoning recorded in its
YAML, per NEXT_STEPS.md's explicit completion condition.

Verified with real Gazebo runs (not synthetic): both pd and lqr paths
through run_clean_experiment.sh still reach stage 4/4 with genuine
results consistent with the already-documented baseline.

Completes private/NEXT_STEPS.md items 3+4+6 as a coherent set. Item 5
(ENV-001, distro comparison) remains separate and not-yet-started.

File: src/double_pendulum_description/urdf/double_pendulum.urdf.xacro (robot description, xacro)
@@ -10,14 +10,23 @@
     which is what Stage A (open-loop check) is supposed to show.
   -->
-  <xacro:property name="m1" value="1.0"/>
-  <xacro:property name="m2" value="1.0"/>
-  <xacro:property name="L1" value="1.0"/>
-  <xacro:property name="L2" value="1.0"/>
-  <xacro:property name="rod_radius" value="0.02"/>
-  <xacro:property name="joint_damping1" value="0.05"/>
-  <xacro:property name="joint_damping2" value="0.05"/>
-  <xacro:property name="tau1_max" value="60.0"/>
-  <xacro:property name="tau2_max" value="30.0"/>
-  <xacro:property name="qd_max" value="50.0"/>
+  <!-- REFACTOR-001: single source of truth is
+       double_pendulum_description/config/plant_params.yaml, also read
+       directly by plant_params.py on the Python/control side, so this
+       xacro and the LQR gain design can never independently drift out
+       of sync (that drift is exactly what SKILL-CONTROL-MODEL-CONSISTENCY
+       existed to guard against as a remembered rule; see
+       harness/skills/retired/ for why it was retired once this made the
+       rule structurally unnecessary). -->
+  <xacro:property name="plant" value="${xacro.load_yaml('../config/plant_params.yaml')}"/>
+  <xacro:property name="m1" value="${plant['m1']}"/>
+  <xacro:property name="m2" value="${plant['m2']}"/>
+  <xacro:property name="L1" value="${plant['L1']}"/>
+  <xacro:property name="L2" value="${plant['L2']}"/>
+  <xacro:property name="rod_radius" value="${plant['rod_radius']}"/>
+  <xacro:property name="joint_damping1" value="${plant['joint_damping1']}"/>
+  <xacro:property name="joint_damping2" value="${plant['joint_damping2']}"/>
+  <xacro:property name="tau1_max" value="${plant['tau1_max']}"/>
+  <xacro:property name="tau2_max" value="${plant['tau2_max']}"/>
+  <xacro:property name="qd_max" value="${plant['qd_max']}"/>
   <material name="base_grey">
     <color rgba="0.35 0.35 0.35 1.0"/>
